File: pcb/kicad_project/m2-fan-controller.kicad_sch (KiCad schematic)
At the start: 0 parts

Commit message: pcb: shcematics + initial component placement
Parts:
- added C1, C2: 0.1uF, Capacitor_SMD:C_0805_2012Metric_Pad1.18x1.45mm_HandSolder, symbol Device:C
- added J1: Bus_M.2_Socket_E, Connector_PCBEdge:M.2_2230-xx-E, symbol Connector:Bus_M.2_Socket_E
- added J2, J3: Conn_01x04, Connector:FanPinHeader_1x04_P2.54mm_Vertical, symbol Connector_Generic:Conn_01x04
- added J4: JST PH_S2B-PH-K, Connector_JST:JST_PH_S2B-PH-K_1x02_P2.00mm_Horizontal, symbol Connector_Generic:Conn_01x02
- added JP1: Jumper_2_Open, Jumper:SolderJumper-2_P1.3mm_Open_RoundedPad1.0x1.5mm, symbol Jumper:Jumper_2_Open
- added R1, R2, R3, R4, R5: 100Ohm, Resistor_SMD:R_0805_2012Metric_Pad1.20x1.40mm_HandSolder, symbol Device:R
- added R6, R7, R8, R9: 10kOhm, Resistor_SMD:R_0805_2012Metric_Pad1.20x1.40mm_HandSolder, symbol Device:R
- added U1: STM32F042F6P6, Package_SO:TSSOP-20_4.4x6.5mm_P0.65mm, symbol MCU_ST_STM32F0:STM32F042F6Px
Connections:
- new net: J1.52 (~{PERST0}), R1.2
- new net: J2.3 (Pin_3), R4.2
- new net: J2.4 (Pin_4), R2.2
- new net: J3.4 (Pin_4), R3.2
- new net: J3.3 (Pin_3), R5.2
- new net +12V: J2.2 (Pin_2), J3.2 (Pin_2), J4.2 (Pin_2)
- new net +3.3V: C1.1, C2.1, J1.2 (3.3V), J1.4 (3.3V), J1.72 (3.3V), J1.74 (3.3V), JP1.1 (A), R6.1, R8.1, R9.1, U1.16 (VDD), U1.5 (VDDA)
- new net BOOT0: JP1.2 (B), R7.1, U1.1 (PB8)
- new net GND: C1.2, C2.2, J1.1 (GND), J1.18 (GND), J1.33 (GND), J1.39 (GND), J1.45 (GND), J1.51 (GND), J1.57 (GND), J1.63 (GND), J1.69 (GND), J1.7 (GND), J1.75 (GND), J2.1 (Pin_1), J3.1 (Pin_1), J4.1 (Pin_1), R7.2, U1.15 (VSSA)
- new net PWM_0: R2.1, U1.12 (PA6)
- new net PWM_1: R3.1, U1.13 (PA7)
- new net RST: R1.1, R6.2, U1.4 (NRST)
- new net TACH_0: R4.1, R8.2, U1.6 (PA0)
- new net TACH_1: R5.1, R9.2, U1.7 (PA1)
- new net USB_D+: J1.3 (USB_D+), U1.18 (PA10/PA12)
- new net USB_D-: J1.5 (USB_D-), U1.17 (PA9/PA11)
- no-connect marks 0 -> 58
Other:
- note added: "Boot config jumper"
- note added: "M.2 connector"
- note added: "MCU"
- note added: "TODO: CHANGE FOOTPRINTS (RIGHT ANGLE)"

Commit message: Hopefully final revision
Parts:
- added TP1: TestPoint, TestPoint:TestPoint_Pad_D1.0mm, symbol Connector:TestPoint
Connections:
- net +3.3V: now also TP1.1
Other:
- note removed: "TODO: CHANGE FOOTPRINTS (RIGHT ANGLE)"
Changed lines of the file:
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@@
-		)
-	)
-	(text "TODO: CHANGE FOOTPRINTS (RIGHT ANGLE)"
-		(exclude_from_sim no)
-		(at 241.808 131.572 0)
-		(effects
-			(font
-				(size 1.27 1.27)
-			)
 		)
 	)
@@
 		(pts
 			(xy 43.18 74.93) (xy 45.72 74.93)
+		)
+		(stroke
+			(width 0)
+			(type default)
+		)
+	)
+	(wire
+		(pts
+			(xy 55.88 162.56) (xy 55.88 165.1)
 		)
 		(stroke
@@
 	)
 	(symbol
+		(lib_id "power:+3.3V")
+		(at 55.88 162.56 0)
+		(unit 1)
+		(exclude_from_sim no)
+		(in_bom yes)
+		(on_board yes)
+		(dnp no)
+		(fields_autoplaced yes)
+		(property "Reference" "#PWR015"
+			(at 55.88 166.37 0)
+			(effects
+				(font
+					(size 1.27 1.27)
+				)
+				(hide yes)
+			)
+		)
+		(property "Value" "+3.3V"
+			(at 55.88 157.48 0)
+			(effects
+				(font
+					(size 1.27 1.27)
+				)
+			)
+		)
+		(property "Footprint" ""
+			(at 55.88 162.56 0)
+			(effects
+				(font
+					(size 1.27 1.27)
+				)
+				(hide yes)
+			)
+		)
+		(property "Datasheet" ""
+			(at 55.88 162.56 0)
+			(effects
+				(font
+					(size 1.27 1.27)
+				)
+				(hide yes)
+			)
+		)
+		(property "Description" "Power symbol creates a global label with name \"+3.3V\""
+			(at 55.88 162.56 0)
+			(effects
+				(font
+					(size 1.27 1.27)
+				)
+				(hide yes)
+			)
+		)
+		(pin "1"
+		)
+		(instances
+			(project ""
+				(path "/827e5d05-dc45-455c-8601-73dd5627afa3"
+					(reference "#PWR015")
+					(unit 1)
+				)
+			)
+		)
+	)
+	(symbol
 		(lib_id "Device:C")
 		(at 149.86 120.65 0)
@@
 					(unit 1)
 				)
+			)
+		)
+	)
+	(symbol
+		(lib_id "Connector:TestPoint")
+		(at 55.88 165.1 180)
+		(unit 1)
+		(exclude_from_sim no)
+		(in_bom yes)
+		(on_board yes)
+		(dnp no)
+		(property "Reference" "TP1"
+			(at 54.61 172.212 0)
+			(effects
+				(font
+					(size 1.27 1.27)
+				)
+				(justify right)
+			)
+		)
+		(property "Value" "TestPoint"
+			(at 58.42 169.6719 0)
+			(effects
+				(font
+					(size 1.27 1.27)
+				)
+				(justify right)
+				(hide yes)
+			)
+		)
+		(property "Footprint" "TestPoint:TestPoint_Pad_D1.0mm"
+			(at 50.8 165.1 0)
+			(effects
+				(font
+					(size 1.27 1.27)
+				)
+				(hide yes)
+			)
+		)
+		(property "Datasheet" "~"
+			(at 50.8 165.1 0)
+			(effects
+				(font
+					(size 1.27 1.27)
+				)
+				(hide yes)
+			)
+		)
+		(property "Description" "test point"
+			(at 55.88 165.1 0)
+			(effects
+				(font
+					(size 1.27 1.27)
+				)
+				(hide yes)
+			)
+		)
+		(pin "1"
+		)
+		(instances
+			(project ""
+				(path "/827e5d05-dc45-455c-8601-73dd5627afa3"
+					(reference "TP1")
+					(unit 1)
+				)

Commit message: Add debug header
Parts:
- removed TP1: TestPoint, TestPoint:TestPoint_Pad_D1.0mm, symbol Connector:TestPoint
- added J5: Conn_02x02_Odd_Even, Connector_PinHeader_2.54mm:PinHeader_1x04_P2.54mm_Vertical, symbol Connector_Generic:Conn_02x02_Odd_Even
- R1, R2, R3, R4, R5, R6, R7, R8, R9: footprint Resistor_SMD:R_0805_2012Metric_Pad1.20x1.40mm_HandSolder -> Resistor_SMD:R_0603_1608Metric_Pad0.98x0.95mm_HandSolder
Connections:
- net +3.3V: now also J5.2 (Pin_2)
- net GND: now also J5.1 (Pin_1)
- net PWM_0: now also U1.13 (PA7); no longer U1.12 (PA6)
- net PWM_1: now also U1.12 (PA6); no longer U1.13 (PA7)
- net SWDIO: now reaches U1.19 (PA13)
- net SWDIO: now also J5.4 (Pin_4)
- net SWCLK: now reaches U1.20 (PA14)
- net SWCLK: now also J5.3 (Pin_3)
- no-connect marks 58 -> 56
Other:
- note added: "Debug header"

Commit message: Final revision
Parts:
- removed JP1: Jumper_2_Open, Jumper:SolderJumper-2_P1.3mm_Open_RoundedPad1.0x1.5mm, symbol Jumper:Jumper_2_Open
- added C3, C4: 0.1uF, Capacitor_SMD:C_0805_2012Metric_Pad1.18x1.45mm_HandSolder, symbol Device:C
- added C5, C6: 1uF, Capacitor_SMD:C_1206_3216Metric, symbol Device:C
- added R10, R11: 10kOhm, Resistor_SMD:R_0603_1608Metric_Pad0.98x0.95mm_HandSolder, symbol Device:R
- added U2, U3: TPS22810DBV, Package_TO_SOT_SMD:SOT-23-6, symbol Power_Management:TPS22810DBV
- C1, C2: footprint Capacitor_SMD:C_0805_2012Metric_Pad1.18x1.45mm_HandSolder -> Capacitor_SMD:C_0603_1608Metric_Pad1.08x0.95mm_HandSolder
- J2, J3: value Conn_01x04 -> JST PH_B4B-PH-K; footprint Connector:FanPinHeader_1x04_P2.54mm_Vertical -> Connector_JST:JST_PH_B4B-PH-K_1x04_P2.00mm_Vertical
- J4: footprint Connector_JST:JST_PH_S2B-PH-K_1x02_P2.00mm_Horizontal -> Connector_JST:JST_PH_B2B-PH-K_1x02_P2.00mm_Vertical
- J5: footprint Connector_PinHeader_2.54mm:PinHeader_1x04_P2.54mm_Vertical -> Connector_PinHeader_1.27mm:PinHeader_1x05_P1.27mm_Vertical; symbol Connector_Generic:Conn_02x02_Odd_Even -> Connector_Generic:Conn_01x05
Connections:
- net +12V: now also C5.1, C6.1, U2.1 (VIN), U3.1 (VIN); no longer J2.2 (Pin_2), J3.2 (Pin_2)
- net +3.3V: now also J5.5 (Pin_5); no longer J5.2 (Pin_2)
- net BOOT0: now also J5.4 (Pin_4)
- net GND: now also C3.2, C4.2, C5.2, C6.2, R10.1, R11.1, U2.2 (GND), U3.2 (GND)
- net SWCLK: now also J5.2 (Pin_2); no longer J5.3 (Pin_3)
- net SWDIO: now also J5.3 (Pin_3); no longer J5.4 (Pin_4)
- net EN_0: now reaches U1.8 (PA2)
- net EN_0: now also R10.2, U2.3 (EN/UVLO)
- net EN_1: now reaches U1.9 (PA3)
- net EN_1: now also R11.2, U3.3 (EN/UVLO)
- new net: C3.1, J2.2 (Pin_2), U2.6 (VOUT)
- new net: C4.1, J3.2 (Pin_2), U3.6 (VOUT)
- no-connect marks 56 -> 58
Other:
- note removed: "Boot config jumper"
- moved on the sheet: C1, C2, J1, J2, J3, J4, R1, R2, R3, R4, R5, R6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

Commit message: Use 0603 components
Parts:
- C3, C4: footprint Capacitor_SMD:C_0805_2012Metric_Pad1.18x1.45mm_HandSolder -> Capacitor_SMD:C_0603_1608Metric_Pad1.08x0.95mm_HandSolder
- C5, C6: footprint Capacitor_SMD:C_1206_3216Metric -> Capacitor_SMD:C_0805_2012Metric_Pad1.18x1.45mm_HandSolder
Changed lines of the file:
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@@
 			)
 		)
-		(property "Footprint" "Capacitor_SMD:C_1206_3216Metric"
+		(property "Footprint" "Capacitor_SMD:C_0805_2012Metric_Pad1.18x1.45mm_HandSolder"
 			(at 150.8252 148.59 0)
 			(effects
@@
 			)
 		)
-		(property "Footprint" "Capacitor_SMD:C_0805_2012Metric_Pad1.18x1.45mm_HandSolder"
+		(property "Footprint" "Capacitor_SMD:C_0603_1608Metric_Pad1.08x0.95mm_HandSolder"
 			(at 199.0852 148.59 0)
 			(effects
@@
 			)
 		)
-		(property "Footprint" "Capacitor_SMD:C_0805_2012Metric_Pad1.18x1.45mm_HandSolder"
+		(property "Footprint" "Capacitor_SMD:C_0603_1608Metric_Pad1.08x0.95mm_HandSolder"
 			(at 199.0852 125.73 0)
 			(effects
@@
 			)
 		)
-		(property "Footprint" "Capacitor_SMD:C_1206_3216Metric"
+		(property "Footprint" "Capacitor_SMD:C_0805_2012Metric_Pad1.18x1.45mm_HandSolder"
 			(at 150.8252 127 0)
 			(effects
