File: pcb/kicad_project/m2-fan-controller.kicad_sch (KiCad schematic)
At the start: 25 parts, among them J1 Bus_M.2_Socket_E, J2 JST PH_B4B-PH-K, J3 JST PH_B4B-PH-K, J4 JST PH_S2B-PH-K, J5 Conn_02x02_Odd_Even, U1 STM32F042F6P6, U2 TPS22810DBV, U3 TPS22810DBV

Commit message: Add 4-ouptut capability + low-frequency PWM control
Parts:
- removed C5, C6: 1uF, Capacitor_SMD:C_0805_2012Metric_Pad1.18x1.45mm_HandSolder, symbol Device:C
- removed R10, R11, R8, R9: 10kOhm, Resistor_SMD:R_0603_1608Metric_Pad0.98x0.95mm_HandSolder, symbol Device:R
- removed R4, R5: 100Ohm, Resistor_SMD:R_0603_1608Metric_Pad0.98x0.95mm_HandSolder, symbol Device:R
- removed U2, U3: TPS22810DBV, Package_TO_SOT_SMD:SOT-23-6, symbol Power_Management:TPS22810DBV
- added D1, D2, D3, D4: GDB5819WS, Diode_SMD:D_SOD-323_HandSoldering, symbol Diode:SS34
- added J4, J5: JST PH_B3B-PH-K, Connector_JST:JST_PH_B3B-PH-K_1x03_P2.00mm_Vertical, symbol Connector_Generic:Conn_01x03
- added NT1: NetTie_2, NetTie:NetTie-2_SMD_Pad0.5mm, symbol Device:NetTie_2
- added Q1, Q3, Q5, Q7: BSS138, Package_TO_SOT_SMD:SOT-23, symbol Transistor_FET:BSS138
- added Q2, Q4, Q6, Q8: AO3401A, Package_TO_SOT_SMD:SOT-23, symbol Transistor_FET:AO3401A
- added R2, R3, R6, R7: 4.7kOhm, Resistor_SMD:R_0603_1608Metric_Pad0.98x0.95mm_HandSolder, symbol Device:R
- added RN1: 1kOhm, Resistor_SMD:R_Array_Convex_4x0603, symbol Device:R_Pack04_Split
- added RN2, RN3: 10kOhm, Resistor_SMD:R_Array_Convex_4x0603, symbol Device:R_Pack04
- added RN4: 100Ohm, Resistor_SMD:R_Array_Convex_4x0603, symbol Device:R_Pack04_Split
- C3, C4: value 0.1uF -> 1uF; footprint Capacitor_SMD:C_0603_1608Metric_Pad1.08x0.95mm_HandSolder -> Capacitor_SMD:C_0805_2012Metric_Pad1.18x1.45mm_HandSolder
- R8: renamed from R2; value 100Ohm -> 1kOhm
- renumbered J5 to J6, J4 to J7, R7 to R4, R6 to R5, R3 to R9
Connections:
- net +12V is gone; now on net 12V: J7.2 (Pin_2)
- net EN_0: now also RN1.3 (R3.1), RN3.6 (R3.2)
- net EN_1: now also RN1.4 (R4.1), RN3.5 (R4.2)
- net GND: now also NT1.2, Q1.2 (S), Q3.2 (S), Q5.2 (S), Q7.2 (S), RN3.1 (R1.1), RN3.2 (R2.1), RN3.3 (R3.1), RN3.4 (R4.1); no longer C3.2, C4.2, J2.1 (Pin_1), J3.1 (Pin_1), J7.1 (Pin_1)
- net TACH_0: now also U1.3 (PF1), RN2.2 (R2.1), RN4.7 (R2.2); no longer U1.6 (PA0)
- net TACH_1: now also U1.10 (PA4), RN2.4 (R4.1), RN4.5 (R4.2); no longer U1.7 (PA1)
- net 12V: now reaches C3.1
- net 12V: now also C4.1, Q2.2 (S), Q4.2 (S), Q6.2 (S), Q8.2 (S), R2.2, R3.2, R6.2, R7.2; no longer J2.2 (Pin_2)
- net at J2.3 (Pin_3): now also RN4.2 (R2.1)
- net TACH_2: now reaches U1.11 (PA5)
- net TACH_2: now also RN2.3 (R3.1), RN4.6 (R3.2)
- net TACH_3: now reaches U1.2 (PF0)
- net TACH_3: now also RN2.1 (R1.1), RN4.8 (R1.2)
- net POWER_1: now reaches J3.2 (Pin_2)
- net POWER_1: now also D2.1 (K), Q4.3 (D); no longer C4.1
- net at J3.3 (Pin_3): now also RN4.4 (R4.1)
- net +3.3V renamed 3V3
- net 3V3: now also RN2.5 (R4.2), RN2.6 (R3.2), RN2.7 (R2.2), RN2.8 (R1.2)
- new net: Q7.1 (G), RN1.7 (R2.2)
- new net: Q7.3 (D), Q8.1 (G), R7.1
- new net: J4.3 (Pin_3), RN4.3 (R3.1)
- new net: Q3.3 (D), Q4.1 (G), R3.1
- new net: Q1.1 (G), RN1.6 (R3.2)
- new net: Q1.3 (D), Q2.1 (G), R2.1
- new net: J5.3 (Pin_3), RN4.1 (R1.1)
- new net: Q5.1 (G), RN1.8 (R1.2)
- new net: Q5.3 (D), Q6.1 (G), R6.1
- new net: Q3.1 (G), RN1.5 (R4.2)
- new net EN_2: RN1.1 (R1.1), RN3.8 (R1.2), U1.6 (PA0)
- new net EN_3: RN1.2 (R2.1), RN3.7 (R2.2), U1.7 (PA1)
- new net FGND: C3.2, C4.2, D1.2 (A), D2.2 (A), D3.2 (A), D4.2 (A), J2.1 (Pin_1), J3.1 (Pin_1), J4.1 (Pin_1), J5.1 (Pin_1), J7.1 (Pin_1), NT1.1
- new net POWER_0: D1.1 (K), J2.2 (Pin_2), Q2.3 (D)
- new net POWER_2: D3.1 (K), J4.2 (Pin_2), Q6.3 (D)
- new net POWER_3: D4.1 (K), J5.2 (Pin_2), Q8.3 (D)
- no-connect marks 58 -> 50
Other:
- note added: "Fan high-side switches"
- note added: "Fan outputs"
- title: (none) -> M.2 Fan Controller
- moved on the sheet: C1, C2, J1, J2, J3, J6, J7, R1, R4, R5, R8, R9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

Commit message: 4 layer layout (#3)
* 4 layer layout

* Final production layout
Parts:
- removed NT1: NetTie_2, NetTie:NetTie-2_SMD_Pad0.5mm, symbol Device:NetTie_2
Connections:
- net FGND is gone; now on net GND: C3.2, C4.2, D1.2 (A), D2.2 (A), D3.2 (A), D4.2 (A), J2.1 (Pin_1), J3.1 (Pin_1), J4.1 (Pin_1), J5.1 (Pin_1), J7.1 (Pin_1)
- net SWCLK: now also J6.3 (Pin_3); no longer J6.2 (Pin_2)
- net SWDIO: now also J6.2 (Pin_2); no longer J6.3 (Pin_3)
Other:
- moved on the sheet: C3, C4, J7

Commit message: Change P-channel mosfets to AO3407A
Parts:
- Q2, Q4, Q6, Q8: value AO3401A -> AO3407A
Changed lines of the file:
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@@
 			)
 		)
-		(property "Value" "AO3401A"
+		(property "Value" "AO3407A"
 			(at 130.81 246.3801 0)
 			(show_name no)
@@
 			)
 		)
-		(property "Value" "AO3401A"
+		(property "Value" "AO3407A"
 			(at 63.5 246.3801 0)
 			(show_name no)
@@
 			)
 		)
-		(property "Value" "AO3401A"
+		(property "Value" "AO3407A"
 			(at 200.66 246.3801 0)
 			(show_name no)
@@
 			)
 		)
-		(property "Value" "AO3401A"
+		(property "Value" "AO3407A"
 			(at 270.51 246.3801 0)
 			(show_name no)
