File: pcb/kicad_project/m2-fan-controller.kicad_pcb (KiCad board)
At the start: 2 copper layers, 30 x 22 mm, 38 parts, among them J1 Bus_M.2_Socket_E, J2 JST PH_B4B-PH-K, J3 JST PH_B4B-PH-K, J4 JST PH_B3B-PH-K, J5 JST PH_B3B-PH-K, J6 Conn_02x02_Odd_Even, J7 JST PH_S2B-PH-K, Q1 BSS138, Q2 AO3401A, Q3 BSS138, Q4 AO3401A, Q5 BSS138, Q6 AO3401A, Q7 BSS138, Q8 AO3401A, U1 STM32F042F6P6

Commit message: 4 layer layout (#3)
* 4 layer layout

* Final production layout
Parts:
- removed NT1: NetTie_2, NetTie:NetTie-2_SMD_Pad0.5mm
- moved C3 6.83 mm to (132.2, 94.3)
- moved C4 6.74 mm to (132.2, 96.3), turned to 180 degrees
- moved RN2 0.85 mm to (133.8, 93.5)
- moved RN4 0.85 mm to (133.8, 96.7)
- moved R1 0.65 mm to (129.1, 95.0)
- moved R5 0.65 mm to (130.7, 95.0), turned to 90 degrees
Connections:
- C3 pad 2: FGND -> GND
- C4 pad 2: FGND -> GND
- D1 pad 2: FGND -> GND
- D2 pad 2: FGND -> GND
- D3 pad 2: FGND -> GND
- D4 pad 2: FGND -> GND
- J2 pad 1: FGND -> GND
- J3 pad 1: FGND -> GND
- J4 pad 1: FGND -> GND
- J5 pad 1: FGND -> GND
- J6 pad 2: /SWCLK -> /SWDIO
- J6 pad 3: /SWDIO -> /SWCLK
- J7 pad 1: FGND -> GND
Routing:
- net FGND: track 84.8 -> 0.00 mm
- net 3V3: track 25.2 -> 45.7 mm
- net GND: track 34.9 -> 18.6 mm, vias 9 -> 17
- net /RST: track 18.6 -> 12.8 mm
- net Net-(J2-Pin_3): track 10.2 -> 7.48 mm
- net /POWER_3: track 7.37 -> 9.03 mm, vias 1 -> 0
- net /TACH_1: track 5.74 -> 7.22 mm
- net /TACH_2: track 15.8 -> 17.2 mm
- net Net-(Q1-G): track 5.49 -> 6.65 mm
- net /TACH_0: track 7.03 -> 8.15 mm
- net /TACH_3: track 8.06 -> 9.16 mm
- net Net-(J3-Pin_3): track 9.45 -> 10.4 mm
- net Net-(J1-~{PERST0}): track 40.3 -> 39.6 mm, vias 3 -> 1
- net /POWER_2: track 9.94 -> 10.6 mm, vias 1 -> 0
- net Net-(J2-Pin_4): track 9.96 -> 9.27 mm
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- added copper zone on B.Cu, net GND
- added copper zone on In1.Cu, net GND
- added copper zone on In2.Cu, net GND
Other:
- copper layers 2 -> 4
- board text removed: "G"
